File: hardware/BLE.kicad_sch (KiCad schematic)
At the start: 4 parts, among them U201 BM832, Y201 32.768KHZ 12.5pF

Commit message: WIP
Other:
- note added: "NINA?"
Changed lines of the file:
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@@
 (kicad_sch (version 20230121) (generator eeschema)
   (paper "A4")
+  (text "NINA?" (at 80.01 53.34 0)
+    (effects (font (size 1.27 1.27)) (justify left bottom))
+  )
   (symbol (lib_id "Device:Crystal_Small") (at 64.77 102.87 0) (unit 1)
     (in_bom yes) (on_board yes) (dnp no) (fields_autoplaced)
