File: hardware/Display.kicad_sch (KiCad schematic)
At the start: 0 parts

Commit message: WIP
Parts:
- added DS1, DS2, DS3, DS4, DS5: LTP-305G, LTP-305G:DIP762W50P254L1875H400Q13, symbol LPLEDSW:LTP-305G
- added DS6: LTP-305G, LPLEDSW:DIP762W50P254L1875H400Q13, symbol LPLEDSW:LTP-305G
